File: battery-pack.kicad_pcb (KiCad board)
At the start: 2 copper layers, 54 parts, among them P1 CONN_01X02, U1 18650-PC8, U2 18650-PC8, U3 18650-PC8, U4 18650-PC8

Commit message: updated schematic
Parts:
- moved D30 26.7 mm to (349.2, 66.7)
- moved D18 24.1 mm to (224.8, 66.7)
- moved D22 22.9 mm to (264.2, 66.7)
- moved R15 22.9 mm to (370.8, 66.7)
- moved R9 21.6 mm to (247.7, 66.7)
- moved D3 21.0 mm to (73.0, 176.5)
- moved R2 21.0 mm to (94.6, 176.5)
- moved R14 21.0 mm to (348.6, 177.8)
- moved D7 20.4 mm to (111.8, 176.5)
- moved R11 20.3 mm to (284.5, 66.7)
- moved R8 20.3 mm to (218.4, 178.4)
- moved D27 20.3 mm to (332.7, 177.8)
- moved R4 19.7 mm to (131.4, 176.5)
- moved D11 19.7 mm to (160.7, 178.4)
- moved R3 19.7 mm to (111.1, 66.7)
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Connections:
- D17 pad 1: Net-(D13-Pad1) -> Net-(D17-Pad1)
- D25 pad 1: Net-(D21-Pad1) -> Net-(D25-Pad1)
- D9 pad 1: Net-(D5-Pad1) -> Net-(D9-Pad1)
- F1 pad 1: Net-(D29-Pad1) -> VCC
- F1 pad 2: Net-(F1-Pad2) -> VCC
- P1 pad 1: Net-(F1-Pad2) -> VCC
- R1 pad 1: Net-(R1-Pad1) -> Net-(D4-Pad1)
- R10 pad 1: Net-(D13-Pad1) -> Net-(D21-Pad1)
- R11 pad 1: Net-(D20-Pad1) -> Net-(D24-Pad1)
- R12 pad 1: Net-(D21-Pad1) -> Net-(D25-Pad1)
- R13 pad 1: Net-(R13-Pad1) -> Net-(D28-Pad1)
- R14 pad 1: Net-(D21-Pad1) -> Net-(D29-Pad1)
- R15 pad 1: Net-(D28-Pad1) -> Net-(D32-Pad1)
- R16 pad 1: Net-(D29-Pad1) -> VCC
- R2 pad 1: GND -> Net-(D5-Pad1)
- R3 pad 1: Net-(D4-Pad1) -> Net-(D8-Pad1)
- R4 pad 1: Net-(D5-Pad1) -> Net-(D9-Pad1)
- R5 pad 1: Net-(R5-Pad1) -> Net-(D12-Pad1)
- R6 pad 1: Net-(D5-Pad1) -> Net-(D13-Pad1)
- R7 pad 1: Net-(D12-Pad1) -> Net-(D16-Pad1)
- R8 pad 1: Net-(D13-Pad1) -> Net-(D17-Pad1)
- R9 pad 1: Net-(R9-Pad1) -> Net-(D20-Pad1)
- U1 pad 2: Net-(R1-Pad1) -> Net-(D4-Pad1)
- U1 pad 3: GND -> Net-(D5-Pad1)
- U1 pad 6: Net-(D4-Pad1) -> Net-(D8-Pad1)
- U1 pad 7: Net-(D5-Pad1) -> Net-(D9-Pad1)
- U2 pad 1: Net-(D5-Pad1) -> Net-(D9-Pad1)
- U2 pad 2: Net-(R5-Pad1) -> Net-(D12-Pad1)
- U2 pad 3: Net-(D5-Pad1) -> Net-(D13-Pad1)
- U2 pad 6: Net-(D12-Pad1) -> Net-(D16-Pad1)
- U2 pad 7: Net-(D13-Pad1) -> Net-(D17-Pad1)
- U3 pad 1: Net-(D13-Pad1) -> Net-(D17-Pad1)
- U3 pad 2: Net-(R9-Pad1) -> Net-(D20-Pad1)
- U3 pad 3: Net-(D13-Pad1) -> Net-(D21-Pad1)
- U3 pad 6: Net-(D20-Pad1) -> Net-(D24-Pad1)
- U3 pad 7: Net-(D21-Pad1) -> Net-(D25-Pad1)
- U4 pad 1: Net-(D21-Pad1) -> Net-(D25-Pad1)
- U4 pad 2: Net-(R13-Pad1) -> Net-(D28-Pad1)
- U4 pad 3: Net-(D21-Pad1) -> Net-(D29-Pad1)
- U4 pad 6: Net-(D28-Pad1) -> Net-(D32-Pad1)
- U4 pad 7: Net-(D29-Pad1) -> VCC
Routing:
- net Net-(D17-Pad1): track 0.00 -> 152.7 mm
- net Net-(D25-Pad1): track 0.00 -> 140.0 mm
- net Net-(D32-Pad1): track 0.00 -> 128.7 mm
- net Net-(D24-Pad1): track 0.00 -> 125.1 mm
- net Net-(D8-Pad1): track 0.00 -> 124.2 mm
- net Net-(D16-Pad1): track 0.00 -> 123.6 mm
- net Net-(D4-Pad1): track 19.0 -> 130.1 mm
- net Net-(D12-Pad1): track 19.0 -> 127.3 mm
- net Net-(D29-Pad1): track 19.1 -> 127.0 mm
- net Net-(D20-Pad1): track 19.1 -> 126.7 mm
- net Net-(D28-Pad1): track 19.1 -> 126.6 mm
- net Net-(D9-Pad1): track 0.00 -> 66.0 mm
- net Net-(D21-Pad1): track 65.5 -> 126.4 mm
- net Net-(D13-Pad1): track 67.6 -> 127.6 mm
- net Net-(D5-Pad1): track 68.7 -> 127.9 mm
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- added copper zone on F.Cu, net VCC
Other:
- board outline added: 362.6 x 134 mm
- net class Default: trace_width 3.048 -> 0.5
- board text added: "60v battery pack version 1.0"
- board text added: "physiii andy@pyfi.org imagination > knowledge"
- board text removed: "imagination > knowledge"
