File: battery-pack.kicad_pcb (KiCad board)
At the start: 2 copper layers, 362.6 x 134 mm, 86 parts, among them P1 CONN_01X02, U1 18650-PC8, U2 18650-PC8, U3 18650-PC8, U4 18650-PC8

Commit message: update
Parts:
- added Q1: MMBT3904LT1G, TO_SOT_Packages_SMD:SOT-23, F.Cu at (86.8, 173.9)
- added Q10: MMBT3904LT1G, TO_SOT_Packages_SMD:SOT-23, F.Cu at (211.9, 173.6)
- added Q11: MMBT3904LT1G, TO_SOT_Packages_SMD:SOT-23, F.Cu at (299.8, 173.3)
- added Q12: MMBT3904LT1G, TO_SOT_Packages_SMD:SOT-23, F.Cu at (382.2, 175.3)
- added Q13: MMBT3904LT1G, TO_SOT_Packages_SMD:SOT-23, F.Cu at (94.5, 67.4)
- added Q14: MMBT3904LT1G, TO_SOT_Packages_SMD:SOT-23, F.Cu at (185.4, 68.4)
- added Q15: MMBT3904LT1G, TO_SOT_Packages_SMD:SOT-23, F.Cu at (270.8, 68.2)
- added Q16: MMBT3904LT1G, TO_SOT_Packages_SMD:SOT-23, F.Cu at (355.1, 67.3)
- added Q2: MMBT3904LT1G, TO_SOT_Packages_SMD:SOT-23, F.Cu at (173.5, 173.8)
- added Q3: MMBT3904LT1G, TO_SOT_Packages_SMD:SOT-23, F.Cu at (261.4, 173.8)
- added Q4: MMBT3904LT1G, TO_SOT_Packages_SMD:SOT-23, F.Cu at (346.4, 174.2)
- added Q5: MMBT3904LT1G, TO_SOT_Packages_SMD:SOT-23, F.Cu at (59.0, 68.0)
- added Q6: MMBT3904LT1G, TO_SOT_Packages_SMD:SOT-23, F.Cu at (146.2, 69.0)
- added Q7: MMBT3904LT1G, TO_SOT_Packages_SMD:SOT-23, F.Cu at (231.6, 68.2)
- added Q8: MMBT3904LT1G, TO_SOT_Packages_SMD:SOT-23, F.Cu at (317.6, 67.3)
- added Q9: MMBT3904LT1G, TO_SOT_Packages_SMD:SOT-23, F.Cu at (124.2, 173.9)
- D1, D13, D14, D15, D16, D17, D18, D19, D2, D20, D29, D3, D30, D31, D32, D4: footprint LEDs:LED-1206 -> LEDs:LED_0805
- D10, D11, D12, D21, D22, D23, D24, D25, D26, D27, D28, D5, D6, D7, D8, D9: footprint LEDs:LED-1206 -> TO_SOT_Packages_SMD:SOT-23
- F1: value FUSE -> 01000057Z; footprint battery-pack:fuse-holder-BK6010 -> battery-pack:ATC_FUSE
- R1, R10, R11, R12, R13, R14, R15, R16, R17, R18, R19, R2, R20, R21, R22, R23, R24, R25, R26, R27, R28, R29, R3, R30, R31, R32, R33, R34, R35, R36, R37, R38, R39, R4, R40, R41, R42, R43, R44, R45, R46, R47, R48, R5, R6, R7, R8, R9: value R -> 10k; footprint Resistors_SMD:R_1206 -> Resistors_SMD:R_0805
- moved R36 281.1 mm to (373.1, 175.2), turned to 90 degrees
- moved R32 271.7 mm to (376.8, 175.1), turned to 90 degrees
- moved R5 251.2 mm to (82.0, 173.7), turned to 270 degrees
- moved R9 242.5 mm to (78.0, 173.7), turned to 90 degrees
- moved R28 237.5 mm to (382.9, 167.8), turned to 270 degrees
- moved R4 225.9 mm to (346.9, 167.6), turned to 270 degrees
- moved D20 225.4 mm to (379.0, 168.1), turned to 90 degrees
- moved R35 222.5 mm to (288.7, 173.3), turned to 90 degrees
- moved D24 221.0 mm to (373.6, 167.9), turned to 180 degrees
- moved R7 220.3 mm to (255.8, 173.8), turned to 90 degrees
- moved R48 218.8 mm to (354.6, 74.5), turned to 270 degrees
- moved R6 211.9 mm to (169.2, 173.8), turned to 270 degrees
- moved R40 195.8 mm to (365.2, 67.3), turned to 90 degrees
- moved R3 195.0 mm to (261.8, 167.5), turned to 270 degrees
- moved R31 193.7 mm to (294.0, 173.3), turned to 90 degrees
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Connections:
- F1 pad 2: VCC -> Net-(F1-Pad2)
- P1 pad 1: VCC -> Net-(F1-Pad2)
- R14 pad 1: Net-(D17-Pad2) -> Net-(D10-Pad2)
- R14 pad 2: Net-(D10-Pad2) -> Net-(D17-Pad2)
- R15 pad 1: Net-(D18-Pad2) -> Net-(D11-Pad2)
- R15 pad 2: Net-(D11-Pad2) -> Net-(D18-Pad2)
- R16 pad 1: Net-(D19-Pad2) -> Net-(D12-Pad2)
- R16 pad 2: Net-(D12-Pad2) -> Net-(D19-Pad2)
- R17 pad 1: Net-(D9-Pad2) -> Net-(Q5-Pad2)
- R17 pad 2: Net-(Q5-Pad2) -> Net-(D9-Pad2)
- R2 pad 1: Net-(D2-Pad1) -> Net-(Q2-Pad1)
- R2 pad 2: Net-(Q2-Pad1) -> Net-(D2-Pad1)
- R21 pad 1: Net-(D13-Pad1) -> Net-(Q5-Pad1)
- R21 pad 2: Net-(Q5-Pad1) -> Net-(D13-Pad1)
- R26 pad 1: Net-(D18-Pad1) -> Net-(Q10-Pad1)
- R26 pad 2: Net-(Q10-Pad1) -> Net-(D18-Pad1)
- R27 pad 1: Net-(D19-Pad1) -> Net-(Q11-Pad1)
- R27 pad 2: Net-(Q11-Pad1) -> Net-(D19-Pad1)
- R28 pad 1: Net-(D20-Pad1) -> Net-(Q12-Pad1)
- R28 pad 2: Net-(Q12-Pad1) -> Net-(D20-Pad1)
- R29 pad 1: Net-(D21-Pad2) -> Net-(Q9-Pad2)
- R29 pad 2: Net-(Q9-Pad2) -> Net-(D21-Pad2)
- R3 pad 1: Net-(D3-Pad1) -> Net-(Q3-Pad1)
- R3 pad 2: Net-(Q3-Pad1) -> Net-(D3-Pad1)
- R30 pad 1: Net-(D22-Pad2) -> Net-(Q10-Pad2)
- R30 pad 2: Net-(Q10-Pad2) -> Net-(D22-Pad2)
- R31 pad 1: Net-(D23-Pad2) -> Net-(Q11-Pad2)
- R31 pad 2: Net-(Q11-Pad2) -> Net-(D23-Pad2)
- R32 pad 1: Net-(D24-Pad2) -> Net-(Q12-Pad2)
- R32 pad 2: Net-(Q12-Pad2) -> Net-(D24-Pad2)
- R37 pad 1: Net-(D1-Pad2) -> Net-(D25-Pad2)
- R37 pad 2: Net-(D25-Pad2) -> Net-(D1-Pad2)
- R38 pad 1: Net-(D2-Pad2) -> Net-(D26-Pad2)
- R38 pad 2: Net-(D26-Pad2) -> Net-(D2-Pad2)
- R39 pad 1: Net-(D3-Pad2) -> Net-(D27-Pad2)
- R39 pad 2: Net-(D27-Pad2) -> Net-(D3-Pad2)
- R4 pad 1: Net-(D4-Pad1) -> Net-(Q4-Pad1)
- R4 pad 2: Net-(Q4-Pad1) -> Net-(D4-Pad1)
- R40 pad 1: Net-(D4-Pad2) -> Net-(D28-Pad2)
- R40 pad 2: Net-(D28-Pad2) -> Net-(D4-Pad2)
- R41 pad 1: Net-(D25-Pad2) -> Net-(Q13-Pad2)
- R41 pad 2: Net-(Q13-Pad2) -> Net-(D25-Pad2)
- R6 pad 1: Net-(D6-Pad2) -> Net-(Q2-Pad2)
- R6 pad 2: Net-(Q2-Pad2) -> Net-(D6-Pad2)
- R7 pad 1: Net-(D7-Pad2) -> Net-(Q3-Pad2)
- R7 pad 2: Net-(Q3-Pad2) -> Net-(D7-Pad2)
- R8 pad 1: Net-(D8-Pad2) -> Net-(Q4-Pad2)
- R8 pad 2: Net-(Q4-Pad2) -> Net-(D8-Pad2)
Routing:
- net Net-(D27-Pad1): track 21.1 -> 144.6 mm
- net Net-(D1-Pad2): track 21.6 -> 142.6 mm
- net Net-(D18-Pad2): track 41.7 -> 160.9 mm
- net Net-(D25-Pad1): track 19.1 -> 138.2 mm
- net Net-(D19-Pad2): track 33.5 -> 151.4 mm
- net Net-(D13-Pad2): track 19.0 -> 136.3 mm
- net Net-(D4-Pad2): track 19.8 -> 136.9 mm
- net Net-(D3-Pad2): track 21.7 -> 138.6 mm
- net Net-(D11-Pad1): track 22.6 -> 139.4 mm
- net Net-(D17-Pad2): track 39.5 -> 155.8 mm
- net Net-(D12-Pad1): track 23.9 -> 140.2 mm
- net Net-(D2-Pad2): track 20.0 -> 136.3 mm
- net Net-(D28-Pad1): track 23.8 -> 139.6 mm
- net Net-(D10-Pad1): track 19.1 -> 133.8 mm
- net Net-(D26-Pad1): track 19.8 -> 134.2 mm
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Other:
- board text added: "Pyfi andy@pyfi.org"
- board text removed: "physiii andy@pyfi.org imagination > knowledge"

Commit message: update
Parts:
- R1, R10, R11, R12, R13, R14, R15, R16, R17, R18, R19, R2, R20, R21, R22, R24, R25, R26, R27, R28, R29, R3, R30, R31, R32, R33, R34, R35, R36, R37, R38, R39, R4, R40, R41, R42, R43, R44, R45, R46, R47, R48, R5, R6, R7, R8, R9: footprint Resistors_SMD:R_0805 -> Resistors_SMD:R_0603
- moved R41 4.96 mm to (105.8, 68.2), turned to 270 degrees
- moved R43 2.70 mm to (278.8, 68.3)
- moved R4 2.52 mm to (347.5, 170.0), turned to 90 degrees
- moved R25 2.19 mm to (125.4, 169.5), turned to 270 degrees
- moved R28 2.13 mm to (383.3, 169.8), turned to 90 degrees
- moved R3 2.11 mm to (262.3, 169.6), turned to 90 degrees
- moved R13 2.07 mm to (65.2, 67.8), turned to 90 degrees
- moved R26 2.07 mm to (212.9, 169.6), turned to 90 degrees
- moved R20 2.02 mm to (324.4, 67.6)
- moved R22 2.02 mm to (145.3, 72.8), turned to 90 degrees
- moved R31 2.00 mm to (292.0, 173.3)
- moved R2 1.92 mm to (174.5, 169.6), turned to 90 degrees
- moved R1 1.88 mm to (87.7, 169.3), turned to 270 degrees
- moved R24 1.82 mm to (316.8, 72.5), turned to 90 degrees
- moved R27 1.78 mm to (300.6, 169.4), turned to 90 degrees
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Routing:
- net Net-(D25-Pad2): track 14.8 -> 7.85 mm
- net Net-(Q13-Pad2): track 4.75 -> 10.7 mm
- net Net-(Q4-Pad1): track 7.43 -> 2.44 mm
- net Net-(Q9-Pad1): track 7.55 -> 2.73 mm
- net Net-(Q12-Pad1): track 8.47 -> 3.69 mm
- net Net-(Q3-Pad1): track 7.22 -> 2.55 mm
- net Net-(Q2-Pad1): track 7.01 -> 2.42 mm
- net Net-(Q10-Pad1): track 6.74 -> 2.25 mm
- net Net-(Q11-Pad1): track 6.65 -> 2.19 mm
- net Net-(Q8-Pad1): track 7.86 -> 3.42 mm
- net Net-(Q15-Pad1): track 7.19 -> 2.75 mm
- net Net-(Q1-Pad1): track 7.10 -> 2.85 mm
- net Net-(Q16-Pad1): track 8.14 -> 4.04 mm
- net Net-(Q6-Pad1): track 5.98 -> 2.10 mm
- net Net-(D27-Pad2): track 12.0 -> 9.05 mm
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