File: _autosave-battery-pack.kicad_pcb (KiCad board)
At the start: 2 copper layers, 362.6 x 134 mm, 86 parts, among them P1 CONN_01X02, U1 18650-PC8, U2 18650-PC8, U3 18650-PC8, U4 18650-PC8

Commit message: update
Parts:
- moved R16 167.6 mm to (297.2, 167.6)
- moved D12 141.9 mm to (257.8, 168.3)
Changed lines of the file:
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@@
   )
   (module LEDs:LED-1206 (layer F.Cu)
-    (at 207.645 35.56)
+    (at 257.81 168.275)
     (descr "LED 1206 smd package")
     (tags "LED1206 SMD")
@@
   )
   (module Resistors_SMD:R_1206 (layer F.Cu)
-    (at 298.45 0)
-    (descr "Resistor SMD 1206, reflow soldering, Vishay (see dcrcw.pdf)")
-    (tags "resistor 1206")
+    (at 297.18 167.64)
+    (descr "Resistor SMD 1206, reflow soldering, Vishay (see dcrcw.pdf)")
+    (tags "resistor 1206")
